File: electronics/BM28B0.6-24DSBreakout/BM28B0.6-24DSBreakout.kicad_pcb (KiCad board)
At the start: 2 copper layers, 15.2 x 35.6 mm, 3 parts, among them J1 Conn_01x14_Male, J2 Conn_01x14_Male, J3 Conn_02x14_Odd_Even

Commit message: Generated gerbers
Other:
- net class Default removed
