File: electronics/LevelShifterBreakout/LevelShifterBreakout.kicad_pcb (KiCad board)
At the start: 2 copper layers, 15.2 x 20.3 mm, 5 parts, among them J1 Conn_01x08_Male, J2 Conn_01x08_Male, U1 SN74AVC4T774RSVR

Commit message: Generated gerbers
Other:
- net class Default removed
- board text added: "~{OE}"
- board text removed: "~OE"
